File: IS-1/ar_long.kicad_sch (KiCad schematic)
At the start: 6 parts

Commit message: update
Parts:
- removed V9: VPULSE, symbol Simulation_SPICE:VPULSE
- added C6: ${SIM.PARAMS}, symbol Device:C
Connections:
- net GND: now also C6.2
- net SIGNAL OUT: now also RV2.3, C6.1; no longer RV2.1
- net at D4.2 (A): now also RV2.1; no longer RV2.3
Other:
- moved on the sheet: C5, RV2

Commit message: ready to pcb
Parts:
- removed C5: ${SIM.PARAMS}, symbol Device:C
Changed lines of the file:
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@@
   (junction (at 154.94 76.2) (diameter 0) (color 0 0 0 0)
   )
-  (junction (at 162.56 76.2) (diameter 0) (color 0 0 0 0)
-  )
   (wire (pts (xy 144.78 83.82) (xy 144.78 76.2))
     (stroke (width 0) (type default))
@@
     (stroke (width 0) (type default))
   )
-  (wire (pts (xy 162.56 76.2) (xy 175.26 76.2))
-    (stroke (width 0) (type default))
-  )
   (wire (pts (xy 110.49 78.74) (xy 110.49 83.82))
     (stroke (width 0) (type default))
@@
     (stroke (width 0) (type default))
   )
-  (wire (pts (xy 162.56 92.71) (xy 162.56 83.82))
-    (stroke (width 0) (type default))
-  )
   (wire (pts (xy 142.24 83.82) (xy 144.78 83.82))
     (stroke (width 0) (type default))
@@
     (stroke (width 0) (type default))
   )
-  (wire (pts (xy 154.94 76.2) (xy 162.56 76.2))
+  (wire (pts (xy 154.94 76.2) (xy 175.26 76.2))
     (stroke (width 0) (type default))
   )
@@
         (path "/733056ea-fa8c-44fe-a8d2-069ece4bafb9/826e54f0-04ab-4e0f-aebf-249b64b4daeb"
           (reference "D4") (unit 1)
-        )
-      )
-    )
-  )
-  (symbol (lib_id "power:GND") (at 162.56 92.71 0) (unit 1)
-    (in_bom yes) (on_board yes) (dnp no) (fields_autoplaced)
-    (property "Reference" "#PWR01" (at 162.56 99.06 0)
-      (effects (font (size 1.27 1.27)) hide)
-    )
-    (property "Value" "GND" (at 162.56 97.79 0)
-      (effects (font (size 1.27 1.27)))
-    )
-    (property "Footprint" "" (at 162.56 92.71 0)
-      (effects (font (size 1.27 1.27)) hide)
-    )
-    (property "Datasheet" "" (at 162.56 92.71 0)
-      (effects (font (size 1.27 1.27)) hide)
-    )
-    (pin "1")
-    (instances
-      (project "IS-1"
-        (path "/733056ea-fa8c-44fe-a8d2-069ece4bafb9/826e54f0-04ab-4e0f-aebf-249b64b4daeb"
-          (reference "#PWR01") (unit 1)
         )
       )
@@
         )
       )
-    )
-  )
-  (symbol (lib_id "Device:C") (at 162.56 80.01 0) (unit 1)
-    (in_bom yes) (on_board yes) (dnp no) (fields_autoplaced)
-    (property "Reference" "C5" (at 166.37 78.74 0)
-      (effects (font (size 1.27 1.27)) (justify left))
-    )
-    (property "Value" "${SIM.PARAMS}" (at 166.37 81.28 0)
-      (effects (font (size 1.27 1.27)) (justify left))
-    )
-    (property "Footprint" "" (at 163.5252 83.82 0)
-      (effects (font (size 1.27 1.27)) hide)
-    )
-    (property "Datasheet" "~" (at 162.56 80.01 0)
-      (effects (font (size 1.27 1.27)) hide)
-    )
-    (property "Sim.Device" "C" (at 162.56 80.01 0)
-      (effects (font (size 1.27 1.27)) hide)
-    )
-    (property "Sim.Type" "=" (at 162.56 80.01 0)
-      (effects (font (size 1.27 1.27)) hide)
-    )
-    (property "Sim.Params" "c=1u" (at 162.56 80.01 0)
-      (effects (font (size 1.27 1.27)) hide)
-    )
-    (property "Sim.Pins" "1=+ 2=-" (at 162.56 80.01 0)
-      (effects (font (size 1.27 1.27)) hide)
-    )
-    (pin "1")
-    (pin "2")
-    (instances
-      (project "IS-1"
-        (path "/733056ea-fa8c-44fe-a8d2-069ece4bafb9/826e54f0-04ab-4e0f-aebf-249b64b4daeb"
-          (reference "C5") (unit 1)
-        )
-      )
